Commit message: Added camera

File: crazyflie_gazebo/models/rotors_description/urdf/component_snippets.xacro (robot description, xacro)
@@ -40,4 +40,77 @@
     </gazebo>
   </xacro:macro>
+  <!-- Macro to add a camera. -->
+  <xacro:macro name="camera_macro"
+    params="namespace parent_link camera_suffix frame_rate
+      horizontal_fov image_width image_height image_format min_distance
+      max_distance noise_mean noise_stddev enable_visual *cylinder *origin">
+    <link name="${namespace}/camera_${camera_suffix}_link">
+      <collision>
+        <origin xyz="0 0 0" rpy="0 0 0" />
+        <geometry>
+          <xacro:insert_block name="cylinder" />
+        </geometry>
+      </collision>
+      <xacro:if value="${enable_visual}">
+        <visual>
+          <origin xyz="0 0 0" rpy="0 1.57079632679 0" />
+          <geometry>
+            <xacro:insert_block name="cylinder" />
+          </geometry>
+          <material name="red" />
+        </visual>
+      </xacro:if>
+      <inertial>
+        <mass value="1e-5" />
+        <origin xyz="0 0 0" rpy="0 0 0" />
+        <inertia ixx="1e-6" ixy="0" ixz="0" iyy="1e-6" iyz="0" izz="1e-6" />
+      </inertial>
+    </link>
+    <joint name="${namespace}/camera_${camera_suffix}_joint" type="fixed">
+      <xacro:insert_block name="origin" />
+      <parent link="${parent_link}" />
+      <child link="${namespace}/camera_${camera_suffix}_link" />
+    </joint>
+    <gazebo reference="${namespace}/camera_${camera_suffix}_link">
+      <sensor type="camera" name="${namespace}_camera_${camera_suffix}">
+        <update_rate>${frame_rate}</update_rate>
+        <camera name="head">
+          <horizontal_fov>${horizontal_fov}</horizontal_fov>
+          <image>
+            <width>${image_width}</width>
+            <height>${image_height}</height>
+            <format>${image_format}</format>
+          </image>
+          <clip>
+            <near>${min_distance}</near>
+            <far>${max_distance}</far>
+          </clip>
+          <noise>
+            <type>gaussian</type>
+            <!-- Noise is sampled independently per pixel on each frame.
+                 That pixel's noise value is added to each of its color
+                 channels, which at that point lie in the range [0,1]. -->
+            <mean>${noise_mean}</mean>
+            <stddev>${noise_stddev}</stddev>
+          </noise>
+        </camera>
+        <plugin name="${namespace}_camera_${camera_suffix}_controller" filename="libgazebo_ros_camera.so">
+          <robotNamespace>${namespace}</robotNamespace>
+          <alwaysOn>true</alwaysOn>
+          <updateRate>${frame_rate}</updateRate>
+          <cameraName>camera_${camera_suffix}</cameraName>
+          <imageTopicName>image_raw</imageTopicName>
+          <cameraInfoTopicName>camera_info</cameraInfoTopicName>
+          <frameName>camera_${camera_suffix}_link</frameName>
+          <hackBaseline>0.0</hackBaseline>
+          <distortionK1>0.0</distortionK1>
+          <distortionK2>0.0</distortionK2>
+          <distortionK3>0.0</distortionK3>
+          <distortionT1>0.0</distortionT1>
+          <distortionT2>0.0</distortionT2>
+        </plugin>
+      </sensor>
+    </gazebo>
+</xacro:macro>
   <!-- Macro to add the controller interface. -->
   <xacro:macro name="controller_plugin_macro" params="namespace imu_sub_topic">

File: crazyflie_gazebo/models/rotors_description/urdf/crazyflie_base.xacro (robot description, xacro)
@@ -44,4 +44,22 @@
         />
   </xacro:if>
+  <!-- Camera -->
+  <xacro:camera_macro
+    namespace="${namespace}"
+    parent_link="base_link"
+    camera_suffix="camera"
+    frame_rate="30.0"
+    horizontal_fov="1.3962634"
+    image_width="800"
+    image_height="800"
+    image_format="R8G8B8"
+    min_distance="0.2"
+    max_distance="300"
+    noise_mean="0.0"
+    noise_stddev="0.007"
+    enable_visual="1" >
+    <box size="0.015 0.02 0.03" />
+    <origin xyz="0.01 0 0.03" rpy="0 0 0" />
+  </xacro:camera_macro>
   <!-- MPU-6500 IMU obtained from  experiments and match datasheets-->
   <xacro:imu_plugin_macro

Commit message: Final

File: crazyflie_gazebo/models/rotors_description/urdf/component_snippets.xacro (robot description, xacro)
@@ -45,5 +45,5 @@
       horizontal_fov image_width image_height image_format min_distance
       max_distance noise_mean noise_stddev enable_visual *cylinder *origin">
-    <link name="${namespace}/camera_${camera_suffix}_link">
+    <link name="${namespace}/${camera_suffix}_link">
       <collision>
         <origin xyz="0 0 0" rpy="0 0 0" />
@@ -67,11 +67,11 @@
       </inertial>
     </link>
-    <joint name="${namespace}/camera_${camera_suffix}_joint" type="fixed">
-      <xacro:insert_block name="origin" />
-      <parent link="${parent_link}" />
-      <child link="${namespace}/camera_${camera_suffix}_link" />
-    </joint>
-    <gazebo reference="${namespace}/camera_${camera_suffix}_link">
-      <sensor type="wideanglecamera" name="${namespace}_camera_${camera_suffix}">
+    <joint name="${namespace}/${camera_suffix}_joint" type="fixed">
+      <xacro:insert_block name="origin" />
+      <parent link="${parent_link}" />
+      <child link="${namespace}/${camera_suffix}_link" />
+    </joint>
+    <gazebo reference="${namespace}/${camera_suffix}_link">
+      <sensor type="camera" name="${camera_suffix}">
         <update_rate>${frame_rate}</update_rate>
         <camera name="head">
@@ -103,12 +103,12 @@
           </lens>
         </camera>
-        <plugin name="${namespace}_camera_${camera_suffix}_controller" filename="libgazebo_ros_camera.so">
+        <plugin name="${namespace}_${camera_suffix}_controller" filename="libgazebo_ros_camera.so">
           <robotNamespace>${namespace}</robotNamespace>
           <alwaysOn>true</alwaysOn>
           <updateRate>${frame_rate}</updateRate>
-          <cameraName>camera_${camera_suffix}</cameraName>
+          <cameraName>${camera_suffix}</cameraName>
           <imageTopicName>image_raw</imageTopicName>
           <cameraInfoTopicName>camera_info</cameraInfoTopicName>
-          <frameName>camera_${camera_suffix}_link</frameName>
+          <frameName>${camera_suffix}_link</frameName>
           <hackBaseline>0.0</hackBaseline>
           <distortionK1>0.0</distortionK1>
