Commit message: Fixed camera placement

File: crazyflie_gazebo/models/rotors_description/urdf/crazyflie_base.xacro (robot description, xacro)
@@ -59,6 +59,6 @@
     noise_stddev="0.007"
     enable_visual="1" >
-    <box size="0.015 0.02 0.03" />
-    <origin xyz="0.01 0 0.03" rpy="0 0 0" />
+    <box size="0.02 0.02 0.02" />
+    <origin xyz="0.01 0 0.02" rpy="0 0 0" />
   </xacro:camera_macro>
   <!-- MPU-6500 IMU obtained from  experiments and match datasheets-->

Commit message: Made it possible to disable/enable camera on Crazyflie

File: crazyflie_gazebo/models/rotors_description/urdf/crazyflie_base.xacro (robot description, xacro)
@@ -27,4 +27,5 @@
   <xacro:property name="use_ros_time" value="$(arg use_ros_time)" />
   <xacro:property name="enable_parameters" value="$(arg enable_parameters)" />
+  <xacro:property name="enable_camera" value="$(arg enable_camera)" />
   <xacro:property name="enable_ground_truth" value="$(arg enable_ground_truth)" />
   <xacro:include filename="$(arg rotors_description_dir)/urdf/component_snippets.xacro"/>
@@ -45,21 +46,23 @@
   </xacro:if>
   <!-- Camera -->
-  <xacro:camera_macro
-    namespace="${namespace}"
-    parent_link="base_link"
-    camera_suffix="camera"
-    frame_rate="60.0"
-    horizontal_fov="1.83259571"
-    image_width="640"
-    image_height="480"
-    image_format="R8G8B8"
-    min_distance="0.2"
-    max_distance="300"
-    noise_mean="0.0"
-    noise_stddev="0.01"
-    enable_visual="1" >
-    <box size="0.02 0.02 0.02" />
-    <origin xyz="0.01 0 0.02" rpy="0 0 0" />
-  </xacro:camera_macro>
+  <xacro:if value="$(arg enable_camera)">
+    <xacro:camera_macro
+      namespace="${namespace}"
+      parent_link="base_link"
+      camera_suffix="camera"
+      frame_rate="60.0"
+      horizontal_fov="1.83259571"
+      image_width="640"
+      image_height="480"
+      image_format="R8G8B8"
+      min_distance="0.2"
+      max_distance="300"
+      noise_mean="0.0"
+      noise_stddev="0.01"
+      enable_visual="1" >
+      <box size="0.02 0.02 0.02" />
+      <origin xyz="0.01 0 0.02" rpy="0 0 0" />
+    </xacro:camera_macro>
+  </xacro:if>
   <!-- MPU-6500 IMU obtained from  experiments and match datasheets-->
   <xacro:imu_plugin_macro

Commit message: Made it possible to change the camera parameters outside of the xacro file

File: crazyflie_gazebo/models/rotors_description/urdf/crazyflie_base.xacro (robot description, xacro)
@@ -28,4 +28,11 @@
   <xacro:property name="enable_parameters" value="$(arg enable_parameters)" />
   <xacro:property name="enable_camera" value="$(arg enable_camera)" />
+  <xacro:property name="camera_fps" value="$(arg camera_fps)" />
+  <xacro:property name="camera_hfov" value="$(arg camera_hfov)" />
+  <xacro:property name="camera_image_width" value="$(arg camera_image_width)" />
+  <xacro:property name="camera_image_height" value="$(arg camera_image_height)" />
+  <xacro:property name="camera_min_distance" value="$(arg camera_min_distance)" />
+  <xacro:property name="camera_max_distance" value="$(arg camera_max_distance)" />
+  <xacro:property name="camera_noise_stddev" value="$(arg camera_noise_stddev)" />
   <xacro:property name="enable_ground_truth" value="$(arg enable_ground_truth)" />
   <xacro:include filename="$(arg rotors_description_dir)/urdf/component_snippets.xacro"/>
@@ -51,13 +58,13 @@
       parent_link="base_link"
       camera_suffix="camera"
-      frame_rate="60.0"
-      horizontal_fov="1.83259571"
-      image_width="640"
-      image_height="480"
+      frame_rate="$(arg camera_fps)"
+      horizontal_fov="$(arg camera_hfov)"
+      image_width="$(arg camera_image_width)"
+      image_height="$(arg camera_image_height)"
       image_format="R8G8B8"
-      min_distance="0.2"
-      max_distance="300"
+      min_distance="$(arg camera_min_distance)"
+      max_distance="$(arg camera_max_distance)"
       noise_mean="0.0"
-      noise_stddev="0.01"
+      noise_stddev="$(arg camera_noise_stddev)"
       enable_visual="1" >
       <box size="0.02 0.02 0.02" />
